File: K_BF.kicad_pcb (KiCad board)
At the start: 2 copper layers, 50 x 50 mm, 23 parts, among them J1 IDC10, J10 SJ1-3535NG, J11 SJ1-3535NG, J12 SJ1-3535NG, J13 SJ1-3535NG, J14 SJ1-3535NG, J9 SJ1-3535NG

Commit message: gerber, silk, schematic added
Parts:
- added G***: LOGO, Cetos:Cetos, B.Cu at (152.5, 49.5)
- added H1: MountingHole_Pad, MountingHole:MountingHole_3.5mm_Pad_Via, F.Cu at (130.1, 86.1)
- moved C7 21.1 mm to (143.5, 75.5), turned to 90 degrees
- moved H2 18.5 mm to (167.0, 86.0)
Routing:
- net Net-(C5-Pad1): track 39.8 -> 49.9 mm, vias 1 -> 2
- net Net-(C7-Pad1): track 21.1 -> 24.5 mm
- net GND: track 0.00 -> 2.48 mm, vias 0 -> 25
- net Net-(J11-Pad5): track 43.4 -> 45.9 mm
- net Net-(J10-Pad5): track 30.7 -> 31.9 mm
- net Net-(J10-Pad4): track 34.6 -> 33.8 mm
- net Net-(C4-Pad1): track 29.6 -> 30.3 mm
Other:
- board text added: "A force d'enculer les poules on finit par casser des œufs."
- board text added: "Je boirai du lait quand les vaches mangeront du raisin"
- board text added: "Kêtos"
- board text added: "La cuvette est pleine de bouillon"
- board text added: "Le Poulpe"
- board text removed: "Cetos"
