File: K_BF.kicad_sch (KiCad schematic)
At the start: 22 parts, among them J1 IDC10, J10 SJ1-3535NG, J11 SJ1-3535NG, J12 SJ1-3535NG, J13 SJ1-3535NG, J14 SJ1-3535NG, J9 SJ1-3535NG

Commit message: gerber, silk, schematic added
Parts:
- added H1: MountingHole_Pad, MountingHole:MountingHole_3.5mm_Pad_Via, symbol Mechanical:MountingHole_Pad
Connections:
- net GND: now also H1.1
Other:
- note added: "A pair of 5W 8 Ohms loudspeakers can be internally plugged on each audio output of the TPA0202. These are differential output (3 Pin J8&J9). Beware to not ground any of the two output wires to avoid destruction of U21"
- note added: "All jack to computer/SDR audio In/out"
- note added: "Kêtos audio dispatching board"
- note added: "Most "Computer Condenser" microphones will work when directly plugged into the MIC connector on the front panel of the Apache Transceiver. The Factory settings for Apache Transceivers is to have a small positive voltage applied to the TIP of the connector for powering a condenser microphone. The RING is connected to push-to-talk, and the SLEEVE is connected to the Transceiver analog ground. The S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"
- note added: "Note : J13 is 100Mb/s. For 1000 Mb/s, no jumper jp5 Mic Bias (see schema) JP6 select ptt if exists P2 is Hermes Altera Jtag for USB Blaster P1 is Altera serial : don't care J15 is Alex J17 Angelia bootloader flash EN (J12 Hermes)"
- note removed: "Schema de principe commutation audio"
- note removed: "To computer/SDR audio In/out"
Changed lines of the file:
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@@
   (no_connect (at 68.58 28.448))
   (no_connect (at 136.906 75.692))
-  (wire (pts (xy 75.946 78.232) (xy 130.556 78.232))
-    (stroke (width 0) (type default))
-  )
   (wire (pts (xy 54.864 121.666) (xy 136.906 121.666))
     (stroke (width 0) (type default))
   )
+  (wire (pts (xy 86.614 78.232) (xy 130.556 78.232))
+    (stroke (width 0) (type default))
+  )
   (wire (pts (xy 68.58 20.828) (xy 69.85 20.828))
     (stroke (width 0) (type default))
@@
     (stroke (width 0) (type default))
   )
-  (wire (pts (xy 55.118 83.566) (xy 75.946 83.566))
+  (wire (pts (xy 86.614 83.566) (xy 86.614 78.232))
     (stroke (width 0) (type default))
   )
@@
     (stroke (width 0) (type default))
   )
-  (wire (pts (xy 77.47 79.502) (xy 156.464 79.502))
-    (stroke (width 0) (type default))
-  )
   (wire (pts (xy 52.832 41.148) (xy 54.102 41.148))
     (stroke (width 0) (type default))
   )
-  (wire (pts (xy 55.118 91.186) (xy 77.47 91.186))
-    (stroke (width 0) (type default))
-  )
-  (wire (pts (xy 75.946 83.566) (xy 75.946 78.232))
+  (wire (pts (xy 98.044 21.844) (xy 98.044 23.114))
     (stroke (width 0) (type default))
   )
@@
     (stroke (width 0) (type default))
   )
+  (wire (pts (xy 99.568 79.502) (xy 156.464 79.502))
+    (stroke (width 0) (type default))
+  )
   (wire (pts (xy 149.606 78.232) (xy 151.384 78.232))
     (stroke (width 0) (type default))
@@
     (stroke (width 0) (type default))
   )
+  (wire (pts (xy 55.118 83.566) (xy 86.614 83.566))
+    (stroke (width 0) (type default))
+  )
   (wire (pts (xy 72.644 63.246) (xy 70.866 63.246))
     (stroke (width 0) (type default))
@@
     (stroke (width 0) (type default))
   )
-  (wire (pts (xy 77.47 91.186) (xy 77.47 79.502))
-    (stroke (width 0) (type default))
-  )
   (wire (pts (xy 70.612 98.806) (xy 71.882 98.806))
     (stroke (width 0) (type default))
@@
     (stroke (width 0) (type default))
   )
+  (wire (pts (xy 55.118 91.186) (xy 99.568 91.186))
+    (stroke (width 0) (type default))
+  )
   (wire (pts (xy 155.956 89.916) (xy 157.226 89.916))
     (stroke (width 0) (type default))
@@
     (stroke (width 0) (type default))
   )
+  (wire (pts (xy 99.568 91.186) (xy 99.568 79.502))
+    (stroke (width 0) (type default))
+  )
   (wire (pts (xy 125.222 73.152) (xy 123.952 73.152))
     (stroke (width 0) (type default))
@@
     (stroke (width 0) (type default))
   )
-  (text "Schema de principe commutation audio" (at 200.152 174.244 0)
-    (effects (font (size 1.27 1.27)) (justify left bottom))
+  (text "Kêtos audio dispatching board\n" (at 200.152 174.244 0)
+    (effects (font (size 2.54 2.54) (thickness 2.54) bold) (justify left bottom))
   )
   (text "internal\n" (at 68.072 140.462 0)
     (effects (font (size 1.27 1.27)) (justify left bottom))
   )
+  (text "Most \"Computer Condenser\" microphones will work when directly plugged into the MIC connector on the front\npanel of the Apache Transceiver. The Factory settings for Apache Transceivers is to have a small positive voltage\napplied to the TIP of the connector for powering a condenser microphone. The RING is connected to\npush-to-talk, and the SLEEVE is connected to the Transceiver analog ground. The SPACE BAR of your\nkeyboard acts as the default push-to-talk for all microphones. A Computer Condenser mic without a push-totalk\nswitch can easily be used by substituting the SPACE BAR of your KEYBOARD."
+    (at 13.462 185.928 0)
+    (effects (font (size 1.27 1.27)) (justify left bottom))
+  )
+  (text "A pair of 5W 8 Ohms loudspeakers can be internally plugged on each audio\noutput of the TPA0202. These are differential output (3 Pin J8&J9). \nBeware to not ground any of the two output wires to avoid destruction \nof U21"
+    (at 12.954 196.088 0)
+    (effects (font (size 1.27 1.27)) (justify left bottom))
+  )
   (text "external\n" (at 34.544 140.462 0)
     (effects (font (size 1.27 1.27)) (justify left bottom))
   )
-  (text "R_hp_out" (at 106.426 78.232 0)
+  (text "R_hp_out" (at 100.838 81.534 0)
     (effects (font (size 1.27 1.27)) (justify left bottom))
   )
@@
     (effects (font (size 2.032 2.032) (thickness 0.4064) bold (color 210 49 255 1)) (justify left bottom))
   )
-  (text "L_hp_out" (at 106.934 81.28 0)
+  (text "L_hp_out" (at 100.838 77.978 0)
+    (effects (font (size 1.27 1.27)) (justify left bottom))
+  )
+  (text "Note : \n\nJ13 is 100Mb/s. For 1000 Mb/s, no jumper\njp5 Mic Bias (see schema)\nJP6 select ptt if exists\nP2 is Hermes Altera Jtag for USB Blaster\nP1 is Altera serial : don't care\nJ15 is Alex\nJ17 Angelia bootloader flash EN (J12 Hermes)\n\n\n\n"
+    (at 130.556 202.438 0)
     (effects (font (size 1.27 1.27)) (justify left bottom))
   )
@@
     (effects (font (size 1.27 1.27) bold) (justify left bottom))
   )
-  (text "To Andromeda \ncontrol panel\n" (at 175.768 63.5 0)
+  (text "To Andromeda \ncontrol panel\n" (at 134.62 64.516 0)
     (effects (font (size 2.54 2.54) (thickness 0.508) bold) (justify left bottom))
   )
-  (text "To computer/SDR \naudio In/out" (at 49.276 151.638 0)
+  (text "All jack \nto computer/SDR \naudio In/out" (at 48.514 141.986 0)
     (effects (font (size 1.27 1.27)) (justify left bottom))
   )
@@
     )
   )
+  (symbol (lib_id "power:GND") (at 98.044 23.114 0) (unit 1)
+    (in_bom yes) (on_board yes) (dnp no) (fields_autoplaced)
+    (property "Reference" "#PWR010" (at 98.044 29.464 0)
+      (effects (font (size 1.27 1.27)) hide)
+    )
+    (property "Value" "GND" (at 98.044 27.2471 0)
+      (effects (font (size 1.27 1.27)))
+    )
+    (property "Footprint" "" (at 98.044 23.114 0)
+      (effects (font (size 1.27 1.27)) hide)
+    )
+    (property "Datasheet" "" (at 98.044 23.114 0)
+      (effects (font (size 1.27 1.27)) hide)
+    )
+    (pin "1")
+    (instances
+      (project "K_BF"
+        (path "/7afd7eec-6096-4a3c-bd88-f2a454a0344e"
+          (reference "#PWR010") (unit 1)
+        )
+      )
+    )
+  )
   (symbol (lib_id "Device:FerriteBead_Small") (at 149.606 87.376 0) (unit 1)
     (in_bom yes) (on_board yes) (dnp no)
@@
         )
       )
+    )
+  )
+  (symbol (lib_id "Mechanical:MountingHole_Pad") (at 98.044 19.304 0) (unit 1)
+    (in_bom yes) (on_board yes) (dnp no) (fields_autoplaced)
+    (property "Reference" "H1" (at 100.584 16.8219 0)
+      (effects (font (size 1.27 1.27)) (justify left))
+    )
+    (property "Value" "MountingHole_Pad" (at 100.584 19.2461 0)
+      (effects (font (size 1.27 1.27)) (justify left) hide)
+    )
+    (property "Footprint" "MountingHole:MountingHole_3.5mm_Pad_Via" (at 98.044 19.304 0)
+      (effects (font (size 1.27 1.27)) hide)
+    )
+    (property "Datasheet" "~" (at 98.044 19.304 0)
+      (effects (font (size 1.27 1.27)) hide)
+    )
+    (pin "1")
+    (instances
+      (project "K_BF"
+        (path "/7afd7eec-6096-4a3c-bd88-f2a454a0344e"
+          (reference "H1") (unit 1)
+        )
+      )
